File: eagle/led_control_v1.0/WS2812B).sch (EAGLE design)
At the start: 30 parts, among them CON2 JACK_DC_BARREL, CON3 SPI, J1 CON_TERMINAL_BLOCK_03-5MM, X2 USB-MICROB, X3 16MHz, X5 22-23-20315.08S

Commit message: Add IR WS2812 code
Other:
- note added: "3 leds to play"
- note added: "I/O"
- note added: "Microcontroller"
- note added: "Power supply"
Changed lines of the file:
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@@
 <text x="205.74" y="99.06" size="5.08" layer="91">ATMega32u4</text>
 <text x="307.34" y="167.64" size="6.4516" layer="91" ratio="5">IR receiver</text>
-<text x="307.34" y="101.6" size="6.4516" layer="91" ratio="5">IR receiver</text>
-<text x="307.34" y="35.56" size="6.4516" layer="91" ratio="5">IR receiver</text>
-<text x="132.08" y="175.26" size="6.4516" layer="91" ratio="5">IR receiver</text>
-<text x="129.54" y="101.6" size="6.4516" layer="91" ratio="5">IR receiver</text>
+<text x="307.34" y="101.6" size="6.4516" layer="91" ratio="5">3 leds to play</text>
+<text x="307.34" y="35.56" size="6.4516" layer="91" ratio="5">I/O</text>
+<text x="132.08" y="175.26" size="6.4516" layer="91" ratio="5">Power supply</text>
+<text x="129.54" y="101.6" size="6.4516" layer="91" ratio="5">Microcontroller</text>
 </plain>
 <instances>
